File: AmeliasHackpad.kicad_sch (KiCad schematic)
At the start: 7 parts, among them SW1 SW_Push, SW2 SW_Push, SW3 SW_Push, SW4 SW_Push, U1 XIAO-RP2040-DIP

Commit message: rotated PCB
Parts:
- added SW5: RotaryEncoder_Switch, Rotary_Encoder:RotaryEncoder_Alps_EC11E-Switch_Vertical_H20mm, symbol Device:RotaryEncoder_Switch
- U1: footprint Module:MOUDLE14P-XIAO-DIP-SMD -> OPL:XIAO-RP2040-DIP
Connections:
- net +5V: no longer D1.2 (VSS), D2.2 (VSS)
- net GND: now also D1.2 (VSS), D2.2 (VSS), SW5.C, SW5.S2; no longer D1.4 (VDD), D2.4 (VDD)
- net at U1.1 (GPIO26/ADC0/A0): now also SW5.A
- net at U1.2 (GPIO27/ADC1/A1): now also SW5.B
- net at U1.3 (GPIO28/ADC2/A2): now also SW5.S1
- new net 5V: D1.4 (VDD), D2.4 (VDD)
